File: pcbs/SM65.kicad_sch (KiCad schematic)
At the start: 43 parts, among them J1 USB_C_Receptacle, J2 Conn_01x03_Pin, U1 AP2112K-3.3TRG1, U2 USBLC6-2SC6, U3 RP2350B, U9 W25Q128JVS, X1 12MHz

Commit message: new branch for rp2350 version
Parts:
- removed C10, C11, C12, C13, C14, C15, C23, C3, C4, C5, C6, C7, C8, C9: 100nF, Mars_Library:C_0402, symbol ProPrj_RP2-easyedapro:UMK105B7104KVHF
- removed C16: 4.7uF, Mars_Library:C_0603, symbol ProPrj_RP2-easyedapro:CL05A475KP5NRNC
- removed C17: 4.7uF, Mars_Library:C_0603, symbol PCM_JLCPCB-Capacitors:0402,4.7uF
- removed C18: 4.7uF, Mars_Library:C_0603, symbol ProPrj_RP2-easyedapro:Device_C
- removed C19: 4.7uF, Mars_Library:C_0603, symbol PCM_JLCPCB-Capacitors:0603,4.7uF
- removed C21, C22: 15pF, Mars_Library:C_0402, symbol EasyEDA:0402CG150J500NT
- removed J2: Conn_01x03_Pin, Connector_PinHeader_2.54mm:PinHeader_1x03_P2.54mm_Vertical, symbol Connector:Conn_01x03_Pin
- removed L1: 3.3uH, Inductor_SMD:L_0805_2012Metric, symbol ProPrj_RP2-easyedapro:AOTA-B201610S3R3-101-T
- removed R4: 33R, Mars_Library:R_0603, symbol ProPrj_RP2-easyedapro:RT0402BRD0733RL
- removed R5: 1R, Mars_Library:R_0603, symbol PCM_JLCPCB-Resistors:0603,1Ω
- removed R6: 200R, Mars_Library:R_0603, symbol PCM_JLCPCB-Resistors:0603,200Ω
- removed R7: 1K, Mars_Library:R_0603, symbol PCM_JLCPCB-Resistors:0603,1kΩ
- removed TP1: TestPoint, TestPoint:TestPoint_Pad_1.0x1.0mm, symbol Connector:TestPoint
- removed U3: RP2350B, RP2350_KiCad:RP2350B_QFN-80_EP_10.573x10.573_Pitch0.4mm, symbol EasyEDA:RP2350B_C42415655
- removed X1: 12MHz, Crystal:Crystal_SMD_3225-4Pin_3.2x2.5mm, symbol ProPrj_RP2-easyedapro:X252012MMB4SI-24
- added C1, C2, C3, C4, C5: 0.1uF, Capacitor_SMD:C_0402_1005Metric_Pad0.74x0.62mm_HandSolder, symbol Mars_Library:C_0.1uF_0402
- added C12, C14: 10uF, Capacitor_SMD:C_0603_1608Metric_Pad1.08x0.95mm_HandSolder, symbol Mars_Library:C_0603
- added C13: 0.1uF, Capacitor_SMD:C_0603_1608Metric_Pad1.08x0.95mm_HandSolder, symbol Mars_Library:C_0603
- added C16, C17: 30p, Capacitor_SMD:C_0603_1608Metric_Pad1.08x0.95mm_HandSolder, symbol Mars_Library:C_0603
- added C6: 1uF, Capacitor_SMD:C_0402_1005Metric_Pad0.74x0.62mm_HandSolder, symbol Mars_Library:C_0.1uF_0402
- added C7, C8: 0.1u, Capacitor_SMD:C_0402_1005Metric_Pad0.74x0.62mm_HandSolder, symbol Mars_Library:C_0.1uF_0402
- added C9: 1u, Capacitor_SMD:C_0402_1005Metric_Pad0.74x0.62mm_HandSolder, symbol Mars_Library:C_0.1uF_0402
- added J2: DEBUG, Mars_Library:SWD_Debug_PinHeader_1x04_P2.54mm, symbol Mars_Library:SWD_Header_4P
- added L1: 10uH, Inductor_SMD:L_0805_2012Metric, symbol Mars_Library:L_10uH_0805
- added R2: 1k_0603, 4ms_Resistor:R_0603, symbol PCM_4ms_Resistor:1k_0603
- added R4, R5: 27R, Resistor_SMD:R_0603_1608Metric_Pad0.98x0.95mm_HandSolder, symbol Mars_Library:R_27R_0603
- added U?: RP2040, Package_DFN_QFN:QFN-56-1EP_7x7mm_P0.4mm_EP3.2x3.2mm, symbol Mars_Library:RP2040
- added Y1: 12MHz, Crystal:Crystal_SMD_3225-4Pin_3.2x2.5mm, symbol Mars_Library:Crystal_12MHz_3225_GND24
- C15: renamed from C20; footprint Mars_Library:C_0402 -> Capacitor_SMD:C_0603_1608Metric_Pad1.08x0.95mm_HandSolder
- renumbered U9 to U3
Connections:
- net +3.3V: now also C1.1, C12.1, C2.1, C3.1, C4.1, C5.1, C6.1, J2.4 (Pin_4), L1.1, R2.1, U?.1 (IOVDD), U?.10 (IOVDD), U?.22 (IOVDD), U?.33 (IOVDD), U?.42 (IOVDD), U?.44 (VREG_IN), U?.48 (USB_VDD), U?.49 (IOVDD)
- net ESD_D+: now also R4.2
- net ESD_D-: now also R5.1
- net GND: now also C1.2, C12.2, C13.2, C14.2, C16.1, C17.1, C2.2, C3.2, C4.2, C5.2, C6.2, C7.2, C8.2, C9.2, J2.1 (Pin_1), U?.19 (TESTEN), U?.57 (GND), Y1.2, Y1.4
- net GPIO0: now also U?.2 (GPIO0)
- net GPIO1: now also U?.3 (GPIO1)
- net GPIO11: now also U?.14 (GPIO11)
- net GPIO12: now also U?.15 (GPIO12)
- net GPIO13: now also U?.16 (GPIO13)
- net GPIO14: now also U?.17 (GPIO14)
- net GPIO15: now also U?.18 (GPIO15)
- net GPIO19: now also U?.30 (GPIO19)
- net GPIO2: now also U?.4 (GPIO2)
- net GPIO20: now also U?.31 (GPIO20)
- net GPIO21: now also U?.32 (GPIO21)
- net GPIO22: now also U?.34 (GPIO22)
- net GPIO23: now also U?.35 (GPIO23)
- net GPIO24: now also U?.36 (GPIO24)
- net GPIO25: now also U?.37 (GPIO25)
- net GPIO26: now also U?.38 (GPIO26_ADC0)
- net GPIO27: now also U?.39 (GPIO27_ADC1)
- net GPIO28: now also U?.40 (GPIO28_ADC2)
- net GPIO29: now also U?.41 (GPIO29_ADC3)
- net GPIO3: now also U?.5 (GPIO3)
- net GPIO4: now also U?.6 (GPIO4)
- net GPIO5: now also U?.7 (GPIO5)
- net GPIO6: now also U?.8 (GPIO6)
- net GPIO7: now also U?.9 (GPIO7)
- net GPIO8: now also U?.11 (GPIO8)
- net GPIO9: now also U?.12 (GPIO9)
- net QPSI_SD3: now also U?.51 (QSPI_SD3)
- net QSPI_SCLK: now also U?.52 (QSPI_SCLK)
- net QSPI_SD0: now also U?.53 (QSPI_SD0)
- net QSPI_SD1: now also U?.55 (QSPI_SD1)
- net QSPI_SD2: now also U?.54 (QSPI_SD2)
- net QSPI_SS: now also R2.2, U?.56 (QSPI_SS)
- net SWCLK: now also J2.2 (Pin_2), U?.24 (SWCLK)
- net SWDIO: now also J2.3 (Pin_3), U?.25 (SWD)
- net RUN: no longer names the net of RUN1.2
- net RUN: now also U?.26 (RUN)
- new net +1V1: C7.1, C8.1, C9.1, U?.23 (DVDD), U?.45 (VREG_VOUT), U?.50 (DVDD)
- new net +3.3VA: C13.1, C14.1, L1.2, U?.43 (ADC_AVDD)
- new net D+: R4.1, U?.47 (USB_DP)
- new net D-: R5.2, U?.46 (USB_DM)
- new net GPIO10: U?.13 (GPIO10)
- new net GPIO16: U?.27 (GPIO16)
- new net GPIO17: U?.28 (GPIO17)
- new net GPIO18: U?.29 (GPIO18)
- new net XIN: C16.2, U?.20 (XIN), Y1.3
- new net XOUT: C17.2, U?.21 (XOUT), Y1.1
Other:
- moved on the sheet: C15, ENC?, RUN1, U3
