File: pcbs/SM65.kicad_sch (KiCad schematic)
At the start: 43 parts, among them J1 USB_C_Receptacle, J2 Conn_01x03_Pin, U1 AP2112K-3.3TRG1, U2 USBLC6-2SC6, U3 RP2350B, U9 W25Q128JVS, X1 12MHz

Commit message: usb enumerated, cdc working to print adc voltages
Parts:
- removed C10, C11, C12, C13, C14, C15, C23, C3, C4, C5, C6, C7, C8, C9: 100nF, Mars_Library:C_0402, symbol ProPrj_RP2-easyedapro:UMK105B7104KVHF
- removed C16: 4.7uF, Mars_Library:C_0603, symbol ProPrj_RP2-easyedapro:CL05A475KP5NRNC
- removed C17: 4.7uF, Mars_Library:C_0603, symbol PCM_JLCPCB-Capacitors:0402,4.7uF
- removed C18: 4.7uF, Mars_Library:C_0603, symbol ProPrj_RP2-easyedapro:Device_C
- removed C19: 4.7uF, Mars_Library:C_0603, symbol PCM_JLCPCB-Capacitors:0603,4.7uF
- removed C21, C22: 15pF, Mars_Library:C_0402, symbol EasyEDA:0402CG150J500NT
- removed J2: Conn_01x03_Pin, Connector_PinHeader_2.54mm:PinHeader_1x03_P2.54mm_Vertical, symbol Connector:Conn_01x03_Pin
- removed L1: 3.3uH, Inductor_SMD:L_0805_2012Metric, symbol ProPrj_RP2-easyedapro:AOTA-B201610S3R3-101-T
- removed R4: 33R, Mars_Library:R_0603, symbol ProPrj_RP2-easyedapro:RT0402BRD0733RL
- removed R5: 1R, Mars_Library:R_0603, symbol PCM_JLCPCB-Resistors:0603,1Ω
- removed R6: 200R, Mars_Library:R_0603, symbol PCM_JLCPCB-Resistors:0603,200Ω
- removed R7: 1K, Mars_Library:R_0603, symbol PCM_JLCPCB-Resistors:0603,1kΩ
- removed TP1: TestPoint, TestPoint:TestPoint_Pad_1.0x1.0mm, symbol Connector:TestPoint
- removed U3: RP2350B, RP2350_KiCad:RP2350B_QFN-80_EP_10.573x10.573_Pitch0.4mm, symbol EasyEDA:RP2350B_C42415655
- removed X1: 12MHz, Crystal:Crystal_SMD_3225-4Pin_3.2x2.5mm, symbol ProPrj_RP2-easyedapro:X252012MMB4SI-24
- added C1, C2, C3, C4, C5: 0.1uF, Capacitor_SMD:C_0402_1005Metric_Pad0.74x0.62mm_HandSolder, symbol Mars_Library:C_0.1uF_0402
- added C12, C14: 10uF, Capacitor_SMD:C_0603_1608Metric_Pad1.08x0.95mm_HandSolder, symbol Mars_Library:C_0603
- added C13: 0.1uF, Capacitor_SMD:C_0603_1608Metric_Pad1.08x0.95mm_HandSolder, symbol Mars_Library:C_0603
- added C16, C17: 30p, Capacitor_SMD:C_0603_1608Metric_Pad1.08x0.95mm_HandSolder, symbol Mars_Library:C_0603
- added C6: 1uF, Capacitor_SMD:C_0402_1005Metric_Pad0.74x0.62mm_HandSolder, symbol Mars_Library:C_0.1uF_0402
- added C7, C8: 0.1u, Capacitor_SMD:C_0402_1005Metric_Pad0.74x0.62mm_HandSolder, symbol Mars_Library:C_0.1uF_0402
- added C9: 1u, Capacitor_SMD:C_0402_1005Metric_Pad0.74x0.62mm_HandSolder, symbol Mars_Library:C_0.1uF_0402
- added J2: DEBUG, Mars_Library:SWD_Debug_PinHeader_1x04_P2.54mm, symbol Mars_Library:SWD_Header_4P
- added L1: 10uH, Inductor_SMD:L_0805_2012Metric, symbol Mars_Library:L_10uH_0805
- added R2: 1k_0603, 4ms_Resistor:R_0603, symbol PCM_4ms_Resistor:1k_0603
- added R4, R5: 27R, Resistor_SMD:R_0603_1608Metric_Pad0.98x0.95mm_HandSolder, symbol Mars_Library:R_27R_0603
- added U4: RP2040, Package_DFN_QFN:QFN-56-1EP_7x7mm_P0.4mm_EP3.2x3.2mm, symbol Mars_Library:RP2040
- added Y1: 12MHz, Crystal:Crystal_SMD_3225-4Pin_3.2x2.5mm, symbol Mars_Library:Crystal_12MHz_3225_GND24
- C15: renamed from C20; footprint Mars_Library:C_0402 -> Capacitor_SMD:C_0603_1608Metric_Pad1.08x0.95mm_HandSolder
- renumbered U9 to U3
Connections:
- net +3.3V: now also C1.1, C12.1, C2.1, C3.1, C4.1, C5.1, C6.1, J2.4 (Pin_4), L1.1, R2.1, U4.1 (IOVDD), U4.10 (IOVDD), U4.22 (IOVDD), U4.33 (IOVDD), U4.42 (IOVDD), U4.44 (VREG_IN), U4.48 (USB_VDD), U4.49 (IOVDD)
- net ESD_D+: now also R4.2
- net ESD_D-: now also R5.1
- net GND: now also C1.2, C12.2, C13.2, C14.2, C16.1, C17.1, C2.2, C3.2, C4.2, C5.2, C6.2, C7.2, C8.2, C9.2, J2.1 (Pin_1), U4.19 (TESTEN), U4.57 (GND), Y1.2, Y1.4
- net GPIO0: now also U4.2 (GPIO0)
- net GPIO1: now also U4.3 (GPIO1)
- net GPIO11: now also U4.14 (GPIO11)
- net GPIO12: now also U4.15 (GPIO12)
- net GPIO13: now also U4.16 (GPIO13)
- net GPIO14: now also U4.17 (GPIO14)
- net GPIO15: now also U4.18 (GPIO15)
- net GPIO19: now also U4.30 (GPIO19)
- net GPIO2: now also U4.4 (GPIO2)
- net GPIO20: now also U4.31 (GPIO20)
- net GPIO21: now also U4.32 (GPIO21)
- net GPIO22: now also U4.34 (GPIO22)
- net GPIO23: now also U4.35 (GPIO23)
- net GPIO24: now also U4.36 (GPIO24)
- net GPIO25: now also U4.37 (GPIO25)
- net GPIO26: now also U4.38 (GPIO26_ADC0)
- net GPIO27: now also U4.39 (GPIO27_ADC1)
- net GPIO28: now also U4.40 (GPIO28_ADC2)
- net GPIO29: now also U4.41 (GPIO29_ADC3)
- net GPIO3: now also U4.5 (GPIO3)
- net GPIO4: now also U4.6 (GPIO4)
- net GPIO5: now also U4.7 (GPIO5)
- net GPIO6: now also U4.8 (GPIO6)
- net GPIO7: now also U4.9 (GPIO7)
- net GPIO8: now also U4.11 (GPIO8)
- net GPIO9: now also U4.12 (GPIO9)
- net QPSI_SD3: now also U4.51 (QSPI_SD3)
- net QSPI_SCLK: now also U4.52 (QSPI_SCLK)
- net QSPI_SD0: now also U4.53 (QSPI_SD0)
- net QSPI_SD1: now also U4.55 (QSPI_SD1)
- net QSPI_SD2: now also U4.54 (QSPI_SD2)
- net QSPI_SS: now also R2.2, U4.56 (QSPI_SS)
- net SWCLK: now also J2.2 (Pin_2), U4.24 (SWCLK)
- net SWDIO: now also J2.3 (Pin_3), U4.25 (SWD)
- net RUN: no longer names the net of RUN1.2
- net RUN: now also U4.26 (RUN)
- new net +1V1: C7.1, C8.1, C9.1, U4.23 (DVDD), U4.45 (VREG_VOUT), U4.50 (DVDD)
- new net +3.3VA: C13.1, C14.1, L1.2, U4.43 (ADC_AVDD)
- new net D+: R4.1, U4.47 (USB_DP)
- new net D-: R5.2, U4.46 (USB_DM)
- new net GPIO10: U4.13 (GPIO10)
- new net GPIO16: U4.27 (GPIO16)
- new net GPIO17: U4.28 (GPIO17)
- new net GPIO18: U4.29 (GPIO18)
- new net XIN: C16.2, U4.20 (XIN), Y1.3
- new net XOUT: C17.2, U4.21 (XOUT), Y1.1
Other:
- moved on the sheet: C15, RUN1, U3

Commit message: improved schematic
Parts:
- removed BOOT1: BOOT, Button_Switch_SMD:SW_SPST_EVQP2_MiddlePushTravel_H2.5mm, symbol Mars_Library:SW_Push_Momentary
- removed C15: 0.1u, Capacitor_SMD:C_0603_1608Metric_Pad1.08x0.95mm_HandSolder, symbol Mars_Library:C_0603
- removed J1: USB_C_Receptacle, Type-C:HRO-TYPE-C-31-M-12, symbol Mars_Library:USB_C_Receptacle_USB2.0_16P
- removed L1: 10uH, Inductor_SMD:L_0805_2012Metric, symbol Mars_Library:L_10uH_0805
- removed R1, R3: 5.1K, Mars_Library:R_0603, symbol Mars_Library:R_5.1k_0603
- removed R2: 1k_0603, 4ms_Resistor:R_0603, symbol PCM_4ms_Resistor:1k_0603
- removed U2: USBLC6-2SC6, Package_TO_SOT_SMD:SOT-23-6, symbol Power_Protection:USBLC6-2SC6
- removed U3: W25Q128JVS, Package_SO:SOIC-8_5.3x5.3mm_P1.27mm, symbol Memory_Flash:W25Q128JVS
- added ANT1: 2.4GHz, Mars_Library:MIFA_2.4GHz_Antenna, symbol Device:Antenna_Shield
- added BOOT1: BOOTSEL, Button_Switch_SMD:SW_SPST_EVQP2_MiddlePushTravel_H2.5mm, symbol Switch:SW_Push
- added C15: 0.1u, Mars_Library:C_0603, symbol Device:C_Small
- added CC1, CC2: 22pF, Mars_Library:C_0402, symbol Mars_Library:C_0402
- added CC3: 2.2nF, Mars_Library:C_0402, symbol Mars_Library:C_0402
- added CC4: 4.7pF, Mars_Library:C_0402, symbol Mars_Library:C_0402
- added CC5: 1.5pF, Mars_Library:C_0402, symbol Mars_Library:C_0402
- added CC6: 1pF, Mars_Library:C_0402, symbol Mars_Library:C_0402
- added CC7: 33nF, Mars_Library:C_0402, symbol Mars_Library:C_0402
- added CC8: 1nF, Mars_Library:C_0402, symbol Mars_Library:C_0402
- added CC9: 10nF, Mars_Library:C_0402, symbol Mars_Library:C_0402
- added FB?: 600R, Mars_Library:Ferrite_0805, symbol Mars_Library:FerriteBead_0805
- added J1: Conn_01x05_Pin, Connector_JST:JST_GH_BM05B-GHS-TBT_1x05-1MP_P1.25mm_Vertical, symbol Connector:Conn_01x05_Pin
- added L1: 8.2nH, symbol Device:L_Small
- added L2: 2.7nH, symbol Device:L_Small
- added L3: 3.9nH, symbol Device:L_Small
- added Q1: AO3401A, Package_TO_SOT_SMD:SOT-23, symbol Transistor_FET:AO3401A
- added Q2: BSS138, Package_TO_SOT_SMD:SOT-23, symbol Mars_Transistor:BSS138
- added R2: 1k, Mars_Library:R_0603, symbol Device:R_Small
- added R3: DNP, Mars_Library:R_0603, symbol Device:R_Small
- added R5: 100K, Mars_Library:R_0603, symbol Device:R_Small
- added R6: 100K, Mars_Library:R_0603, symbol Mars_Library:R_0603
- added R7: 1M, Mars_Library:R_0603, symbol Device:R_Small
- added RR1: 1M, Mars_Library:R_0402, symbol Mars_Library:R_0402
- added RR2: 22K, Mars_Library:R_0402, symbol Mars_Library:R_0402
- added U2: W25Q128JVS, Package_SO:SOIC-8_5.3x5.3mm_P1.27mm, symbol Memory_Flash:W25Q128JVS
- added U3: SN74LV1T125DBV, Package_TO_SOT_SMD:SOT-23-5, symbol Logic_LevelTranslator:SN74LV1T125DBV
- added U5: MCP3208, Package_SO:SOIC-16_3.9x9.9mm_P1.27mm, symbol Analog_ADC:MCP3208
- added U?: nRF24L01P, Package_DFN_QFN:QFN-20-1EP_4x4mm_P0.5mm_EP2.5x2.5mm, symbol RF:nRF24L01P
- added Y?: 16MHz, symbol Device:Crystal_GND24_Small
- J2: footprint Mars_Library:SWD_Debug_PinHeader_1x04_P2.54mm -> Connector_PinHeader_1.27mm:PinHeader_1x04_P1.27mm_Vertical
- gave numbers to parts that had none: 1
- renumbered C7 to C1, C12 to C10, C13 to C11, C14 to C12, C1 to C13, C2 to C14, C8 to C2, C9 to C3, C1 to C4, C2 to C5, C3 to C6, C4 to C7, C5 to C8, C6 to C9, R4 to R1, R5 to R4
Connections:
- net ESD_D+ is gone; now on net D+: R1.2
- net ESD_D- is gone; now on net D-: R4.1
- net GPIO7 is gone; now on net ENC_A_GP7: U4.9 (GPIO7)
- net GPIO8 is gone; now on net ENC_B_GP8: U4.11 (GPIO8)
- net GPIO9 is gone; now on net ENC_SW_GP9: U4.12 (GPIO9)
- net +3.3V: now also CC8.1, CC9.1, FB?.1, U?.15 (VDD), U?.18 (VDD), U?.7 (VDD)
- net +3.3VA: now also FB?.2, U5.15 (Vref), U5.16 (Vdd)
- net +5V: now also Q1.3 (D); no longer C13.1, FB1.2, U1.1 (IN), U1.3 (EN)
- net D+: now also J1.4 (Pin_4); no longer R1.1, U4.47 (USB_DP)
- net D-: now also J1.3 (Pin_3); no longer R4.2, U4.46 (USB_DM)
- net GND: now also ANT1.2 (Shield), BOOT1.1, C15.2, CC1.2, CC2.2, CC3.2, CC4.2, CC6.2, CC7.2, CC8.2, CC9.2, J1.5 (Pin_5), Q2.2 (S), R7.1, RR2.1, U2.4 (GND), U3.1 (~{OE}), U3.3 (GND), U5.14 (AGND), U5.9 (DGND), U?.14 (VSS), U?.17 (VSS), U?.20 (VSS), U?.8 (VSS), Y?.2, Y?.4
- net QSPI_SCLK: now also U2.6 (CLK)
- net QSPI_SD0: now also U2.5 (DI/IO_{0})
- net QSPI_SD1: now also U2.2 (DO/IO_{1})
- net QSPI_SD2: now also U2.3 (~{WP}/IO_{2})
- net QSPI_SS: now also R2.1, R3.1, U2.1 (~{CS})
- net VBUS: now also J1.2 (Pin_2)
- net ENC_A_GP16 renamed ENC_A_GP7
- net ENC_B_GP17 renamed ENC_B_GP8
- net ENC_SW_GP18 renamed ENC_SW_GP9
- net GPIO10: no longer names the net of U4.13 (GPIO10)
- net GPIO11: no longer names the net of U4.14 (GPIO11)
- net GPIO12: no longer names the net of U4.15 (GPIO12)
- net GPIO13: no longer names the net of U4.16 (GPIO13)
- net GPIO16 renamed ADC_DOUT/MISO
- net GPIO17 renamed ADC_CS
- net GPIO18 renamed ADC_CLK
- net GPIO19 renamed ADC_DIN/MOSI
- net GPIO2 renamed MUX_S0
- net GPIO22 renamed 3V_RGB
- net 3V_RGB: now also U3.2 (A)
- net GPIO23 renamed GP23_LED_EN
- net GP23_LED_EN: now also R6.1
- net GPIO3 renamed MUX_S1
- net GPIO4 renamed MUX_S2
- net GPIO5 renamed MUX_S3
- new net: L1.1, L2.1, U?.12 (ANT1)
- new net: L1.2, L3.2, U?.13 (ANT2)
- new net: CC2.1, RR1.2, U?.9 (XC2), Y?.1
- new net: CC1.1, RR1.1, U?.10 (XC1), Y?.3
- new net: CC3.1, CC4.1, L2.2, U?.11 (VDD_PA)
- new net: CC7.1, U?.19 (DVDD)
- new net: RR2.2, U?.16 (IREF)
- new net: CC5.2, L3.1
- new net +3V3: C15.1, R3.2, U2.8 (VCC)
- new net +5V_RAW: C13.1, FB1.2, Q1.2 (S), R5.2, U1.1 (IN), U1.3 (EN), U3.5 (VCC)
- new net 50ohm: ANT1.1 (A), CC5.1, CC6.1
- new net 5V_RGB_OUT: U3.4 (Y)
- new net ADC_CH0: U5.1 (CH0)
- new net ADC_CH1: U5.2 (CH1)
- new net ADC_CH2: U5.3 (CH2)
- new net ADC_CH3: U5.4 (CH3)
- new net ADC_CH4: U5.5 (CH4)
- new net GPIO16_DOUT/MISO: U5.12 (Dout)
- new net GPIO17_CS: U5.10 (~{CS}/SHDN)
- new net GPIO18_CLK: U5.13 (CLK)
- new net GPIO19_DIN/MOSI: U5.11 (Din)
- new net LED_GATE: Q2.1 (G), R6.2, R7.2
- new net NRF_CE: U?.1 (CE)
- new net NRF_CLK: U?.3 (SCK)
- new net NRF_CS: U?.2 (CSN)
- new net NRF_IRQ: U?.6 (IRQ)
- new net NRF_MISO: U?.5 (MISO)
- new net NRF_MOSI: U?.4 (MOSI)
- new net N_DRAIN_5V: Q1.1 (G), Q2.3 (D), R5.1
- new net QSPI_SD3: U2.7 (~{HOLD}/~{RESET}/IO_{3})
- new net R_D+: R1.1, U4.47 (USB_DP)
- new net R_D-: R4.2, U4.46 (USB_DM)
- new net USB_BOOT: BOOT1.2, R2.2
- new net VBAT: J1.1 (Pin_1)
- no-connect marks 2 -> 0
Other:
- sheet lighting ports: added LED_IN; removed none
- sheet sensors ports: added MUX1, MUX2, MUX3, MUX4, MUX5, MUX_S0, MUX_S1, MUX_S2, MUX_S3; removed none
- note added: "3.3V > 5V level shifter"
- note added: "5V pullup, active LOW"
- note added: "Flash + Boot"
- note added: "LED 5V rail transistor"
- moved on the sheet: C1, C10, C11, C12, C13, C14, C16, C17, C2, C3, C4, C5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

Commit message: pcb updated
Parts:
- added D1, D2: SS14, Diode_SMD:D_SMA, symbol Device:D_Schottky_Small
- added D3: RED, LED_SMD:LED_0402_1005Metric, symbol Device:LED_Small
- added Q3: BSS138, Package_TO_SOT_SMD:SOT-23, symbol Mars_Transistor:BSS138
- added R10, R14, R15, R9: 100K, Mars_Library:R_0603, symbol Mars_Library:R_0603
- added R11: 1M, Mars_Library:R_0603, symbol Device:R_Small
- added R12: 10K, Mars_Library:R_0402, symbol Mars_Library:R_0402
- added R13: 2K, Mars_Library:R_0603, symbol Mars_Library:R_0603
- added SW1: MS-22D18G2ROHS, MS-22D18G2ROHS:MS-22D18_SMD, symbol MS-22D18G2ROHS:MS-22D18G2ROHS
- added U12: TP4056-42-ESOP8, Package_SO:SOIC-8-1EP_3.9x4.9mm_P1.27mm_EP2.41x3.3mm, symbol Battery_Management:TP4056-42-ESOP8
- C1, C2, C3, C4, C5, C6, C7, C8, C9: footprint Capacitor_SMD:C_0402_1005Metric_Pad0.74x0.62mm_HandSolder -> Mars_Library:C_0402
- C10, C11, C12: footprint Capacitor_SMD:C_0603_1608Metric_Pad1.08x0.95mm_HandSolder -> Mars_Library:C_0603
- C16, C17: footprint Capacitor_SMD:C_0603_1608Metric_Pad1.08x0.95mm_HandSolder -> Mars_Library:C_0402
- FB2: renamed from FB?; footprint Mars_Library:Ferrite_0805 -> PCM_Ferrite_SMD_AKL:Ferrite_0603_1608Metric
- J1: value Conn_01x05_Pin -> Daughter
- L1, L2, L3: footprint (none) -> Mars_Library:R_0402
- Y2: renamed from Y?; footprint (none) -> Crystal:Crystal_SMD_3225-4Pin_3.2x2.5mm
- gave numbers to parts that had none: 1
Connections:
- net +3V3 is gone; now on net +3.3V: C15.1, R3.2, U2.8 (VCC)
- net GPIO14 is gone; now on net NRF_CE: U4.17 (GPIO14)
- net GPIO15 is gone; now on net NRF_IRQ: U4.18 (GPIO15)
- net GPIO16_DOUT/MISO is gone; now on net ADC_DOUT/MISO: U5.12 (Dout)
- net GPIO17_CS is gone; now on net ADC_CS: U5.10 (~{CS}/SHDN)
- net GPIO18_CLK is gone; now on net ADC_CLK: U5.13 (CLK)
- net GPIO19_DIN/MOSI is gone; now on net ADC_DIN/MOSI: U5.11 (Din)
- net NRF_CS is gone; now on net NRF_CSN: U11.2 (CSN)
- net QPSI_SD3 is gone; now on net QSPI_SD3: U4.51 (QSPI_SD3)
- net +5V_RAW: now also D1.2 (A), R9.2, U12.4 (V_{CC}); no longer C13.1, Q1.2 (S), R5.2, U1.1 (IN), U1.3 (EN), U3.5 (VCC)
- net GND: now also Q3.2 (S), R11.1, R12.2, R13.2, R15.1, SW1.4, U12.1 (TEMP), U12.3 (GND), U12.9 (EPAD)
- net NRF_CLK: now also U4.13 (GPIO10)
- net NRF_MISO: now also U4.15 (GPIO12)
- net NRF_MOSI: now also U4.14 (GPIO11)
- net NRF_CSN: now reaches U4.16 (GPIO13)
- net BAT_VOLTAGE: now reaches U5.8 (CH7)
- net BAT_VOLTAGE: now also R14.2, R15.2
- net GPIO20 renamed SW_STATUS_GP20
- net SW_STATUS_GP20: now also SW1.5
- net GPIO24 renamed BAT_CE
- net BAT_CE: now also R10.1
- net VBAT renamed BAT+
- net BAT+: now also R14.1, SW1.3, U12.5 (BAT)
- new net: D3.1 (K), R12.1
- new net: R13.1, U12.2 (PROG)
- new net BAT_GATE: Q3.1 (G), R10.2, R11.2
- new net BAT_SW: D2.2 (A), SW1.2
- new net PWR_IN: C13.1, D1.1 (K), D2.1 (K), Q1.2 (S), R5.2, U1.1 (IN), U1.3 (EN), U3.5 (VCC)
- new net R_BAT_CE: Q3.3 (D), R9.1, U12.8 (CE)
- new net R_CHRG: D3.2 (A), U12.7 (~{CHRG})
- no-connect marks 0 -> 2
Other:
- sheet lighting ports: added RGB_IN; removed LED_IN
- note added: "3.3V Regulator"
- note added: "3.3VA Filtering"
- note added: "Analog and ADC"
- note added: "Battery Charging and Power Switch"
- note added: "Daughterboard Connect"
- note added: "Main MCU"
- note added: "Power Rails"
- note added: "Power and Voltage Regulation"
- note added: "Rotary Encoder"
- note added: "nRF24L01 Radio Circuit"
- moved on the sheet: ANT1, BOOT1, C1, C13, C14, C15, C16, C17, C2, C3, C4, C5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
