File: pcbs/lighting.kicad_sch (KiCad schematic)
At the start: 68 parts

Commit message: improved schematic
Parts:
- added C23, C24, C25, C26, C27, C28, C29, C30, C31, C32, C33, C34, C35, C36, C37, C38, C39, C40, C41, C42, C43, C44, C45, C46, C47, C48, C49, C50, C51, C52, C53, C54, C55, C56, C57, C58, C59, C60, C61, C62, C63, C64, C65, C66, C67, C68, C69, C70, C71, C72, C73, C74, C75, C76, C77, C78, C79, C80, C81, C82, C83, C84, C85, C86, C87, C88, C89, C90: C, Mars_Library:C_0402, symbol Mars_Library:C_0402
- gave numbers to parts that had none: 3
- renumbered LED0 to LED1, LED9 to LED10, LED10 to LED11, LED11 to LED12, LED12 to LED13, LED13 to LED14, LED14 to LED15, LED15 to LED16, LED16 to LED17, LED17 to LED18, LED18 to LED19, LED1 to LED2, LED19 to LED20, LED20 to LED21, LED21 to LED22, LED22 to LED23, LED23 to LED24, LED24 to LED25, LED25 to LED26, LED26 to LED27, LED27 to LED28, LED28 to LED29, LED2 to LED3, LED29 to LED30, LED30 to LED31, LED31 to LED32, LED32 to LED33, LED33 to LED34, LED34 to LED35, LED35 to LED36, LED36 to LED37, LED37 to LED38, LED38 to LED39, LED3 to LED4, LED39 to LED40, LED40 to LED41, LED41 to LED42, LED42 to LED43, LED43 to LED44, LED44 to LED45, LED45 to LED46, LED46 to LED47, LED47 to LED48, LED48 to LED49, LED4 to LED5, LED49 to LED50, LED50 to LED51, LED51 to LED52, LED52 to LED53, LED53 to LED54, LED54 to LED55, LED55 to LED56, LED56 to LED57, LED57 to LED58, LED58 to LED59, LED5 to LED6, LED59 to LED60, LED60 to LED61, LED61 to LED62, LED62 to LED63, LED63 to LED64, LED6 to LED7, LED7 to LED8, LED8 to LED9, R2 to R8
Connections:
- net LED_GP10 is gone; now on net LED_IN: R8.1
- net +5V: now also C23.1, C24.1, C25.1, C26.1, C27.1, C28.1, C29.1, C30.1, C31.1, C32.1, C33.1, C34.1, C35.1, C36.1, C37.1, C38.1, C39.1, C40.1, C41.1, C42.1, C43.1, C44.1, C45.1, C46.1, C47.1, C48.1, C49.1, C50.1, C51.1, C52.1, C53.1, C54.1, C55.1, C56.1, C57.1, C58.1, C59.1, C60.1, C61.1, C62.1, C63.1, C64.1, C65.1, C66.1, C67.1, C68.1, C69.1, C70.1, C71.1, C72.1, C73.1, C74.1, C75.1, C76.1, C77.1, C78.1, C79.1, C80.1, C81.1, C82.1, C83.1, C84.1, C85.1, C86.1, C87.1, C88.1, C89.1, C90.1
- net GND: now also C23.2, C24.2, C25.2, C26.2, C27.2, C28.2, C29.2, C30.2, C31.2, C32.2, C33.2, C34.2, C35.2, C36.2, C37.2, C38.2, C39.2, C40.2, C41.2, C42.2, C43.2, C44.2, C45.2, C46.2, C47.2, C48.2, C49.2, C50.2, C51.2, C52.2, C53.2, C54.2, C55.2, C56.2, C57.2, C58.2, C59.2, C60.2, C61.2, C62.2, C63.2, C64.2, C65.2, C66.2, C67.2, C68.2, C69.2, C70.2, C71.2, C72.2, C73.2, C74.2, C75.2, C76.2, C77.2, C78.2, C79.2, C80.2, C81.2, C82.2, C83.2, C84.2, C85.2, C86.2, C87.2, C88.2, C89.2, C90.2

Commit message: pcb updated
Parts:
- removed C24, C25, C26, C27, C28, C29, C30, C31, C32, C33, C34, C35, C36, C37, C38, C39, C40, C41, C42, C43, C44, C45, C46, C47, C48, C49, C50, C51, C52, C53, C54, C55, C56, C57, C58, C59, C60, C61, C62, C63, C64, C65, C66, C67, C68, C69, C70, C71, C72, C73, C74, C75, C76, C77, C78, C79, C80, C81, C82, C83, C84, C85, C86, C87, C88, C89, C90: C, Mars_Library:C_0402, symbol Mars_Library:C_0402
- added LC10, LC11, LC12, LC13, LC14, LC15, LC16, LC17, LC18, LC19, LC2, LC20, LC21, LC22, LC23, LC24, LC25, LC26, LC27, LC28, LC29, LC3, LC30, LC31, LC32, LC33, LC34, LC35, LC36, LC37, LC38, LC39, LC4, LC40, LC41, LC42, LC43, LC44, LC45, LC46, LC47, LC48, LC49, LC5, LC50, LC51, LC52, LC53, LC54, LC55, LC56, LC57, LC58, LC59, LC6, LC60, LC61, LC62, LC63, LC64, LC65, LC66, LC67, LC68, LC7, LC8, LC9: 0.1uF, Mars_Library:C_0402, symbol Mars_Library:C_0402
- added LED68: SK6812MINI-E, PCM_marbastlib-various:LED_6028R, symbol PCM_marbastlib-various:SK6812MINI-E
- LC1: renamed from C23; value C -> 0.1uF
Connections:
- net +5V: now also LC10.1, LC11.1, LC12.1, LC13.1, LC14.1, LC15.1, LC16.1, LC17.1, LC18.1, LC19.1, LC2.1, LC20.1, LC21.1, LC22.1, LC23.1, LC24.1, LC25.1, LC26.1, LC27.1, LC28.1, LC29.1, LC3.1, LC30.1, LC31.1, LC32.1, LC33.1, LC34.1, LC35.1, LC36.1, LC37.1, LC38.1, LC39.1, LC4.1, LC40.1, LC41.1, LC42.1, LC43.1, LC44.1, LC45.1, LC46.1, LC47.1, LC48.1, LC49.1, LC5.1, LC50.1, LC51.1, LC52.1, LC53.1, LC54.1, LC55.1, LC56.1, LC57.1, LC58.1, LC59.1, LC6.1, LC60.1, LC61.1, LC62.1, LC63.1, LC64.1, LC65.1, LC66.1, LC67.1, LC68.1, LC7.1, LC8.1, LC9.1, LED68.1 (VDD)
- net GND: now also LC10.2, LC11.2, LC12.2, LC13.2, LC14.2, LC15.2, LC16.2, LC17.2, LC18.2, LC19.2, LC2.2, LC20.2, LC21.2, LC22.2, LC23.2, LC24.2, LC25.2, LC26.2, LC27.2, LC28.2, LC29.2, LC3.2, LC30.2, LC31.2, LC32.2, LC33.2, LC34.2, LC35.2, LC36.2, LC37.2, LC38.2, LC39.2, LC4.2, LC40.2, LC41.2, LC42.2, LC43.2, LC44.2, LC45.2, LC46.2, LC47.2, LC48.2, LC49.2, LC5.2, LC50.2, LC51.2, LC52.2, LC53.2, LC54.2, LC55.2, LC56.2, LC57.2, LC58.2, LC59.2, LC6.2, LC60.2, LC61.2, LC62.2, LC63.2, LC64.2, LC65.2, LC66.2, LC67.2, LC68.2, LC7.2, LC8.2, LC9.2, LED68.4 (VSS)
- net at LED67.2 (DOUT): now also LED68.3 (DIN)
- net LED_IN renamed LED_DIN
- net LED_DIN: no longer R8.1
- new net RGB_IN: R8.1
Other:
- moved on the sheet: LC1
