File: pcbs/sensors.kicad_sch (KiCad schematic)
At the start: 69 parts

Commit message: improved schematic
Parts:
- removed U?: ADG732BSUZ, ADG732BSUZ:QFP50P900X900X120-49N, symbol ADG732BSUZ:ADG732BSUZ
- added C18, C19, C20, C21, C22: C, Mars_Library:C_0402, symbol Mars_Library:C_0402
- added U10, U6, U7, U8, U9: CD74HC4067SM, Package_SO:SSOP-24_5.3x8.2mm_P0.65mm, symbol 74xx:CD74HC4067SM
- renumbered HE0 to HE1, HE9 to HE10, HE10 to HE11, HE11 to HE12, HE12 to HE13, HE13 to HE14, HE14 to HE15, HE15 to HE16, HE16 to HE17, HE17 to HE18, HE18 to HE19, HE1 to HE2, HE19 to HE20, HE20 to HE21, HE21 to HE22, HE22 to HE23, HE23 to HE24, HE24 to HE25, HE25 to HE26, HE26 to HE27, HE27 to HE28, HE28 to HE29, HE2 to HE3, HE29 to HE30, HE30 to HE31, HE31 to HE32, HE32 to HE33, HE33 to HE34, HE34 to HE35, HE35 to HE36, HE36 to HE37, HE37 to HE38, HE38 to HE39, HE3 to HE4, HE39 to HE40, HE40 to HE41, HE41 to HE42, HE42 to HE43, HE43 to HE44, HE44 to HE45, HE45 to HE46, HE46 to HE47, HE47 to HE48, HE48 to HE49, HE4 to HE5, HE49 to HE50, HE50 to HE51, HE51 to HE52, HE52 to HE53, HE53 to HE54, HE54 to HE55, HE55 to HE56, HE56 to HE57, HE57 to HE58, HE58 to HE59, HE5 to HE6, HE59 to HE60, HE60 to HE61, HE61 to HE62, HE62 to HE63, HE63 to HE64, HE64 to HE65, HE65 to HE66, HE66 to HE67, HE67 to HE68, HE6 to HE7, HE7 to HE8, HE8 to HE9
Connections:
- net +3.3V: now also C18.1, C19.1, C20.1, C21.1, C22.1, U10.24 (VCC), U6.24 (VCC), U7.24 (VCC), U8.24 (VCC), U9.24 (VCC)
- net GND: now also C18.2, C19.2, C20.2, C21.2, C22.2, U10.12 (GND), U10.15 (~{E}), U6.12 (GND), U6.15 (~{E}), U7.12 (GND), U7.15 (~{E}), U8.12 (GND), U8.15 (~{E}), U9.12 (GND), U9.15 (~{E})
- new net MUX1: U6.1 (COM)
- new net MUX2: U7.1 (COM)
- new net MUX3: U8.1 (COM)
- new net MUX4: U9.1 (COM)
- new net MUX5: U10.1 (COM)
- new net MUX_S0: U10.10 (S0), U6.10 (S0), U7.10 (S0), U8.10 (S0), U9.10 (S0)
- new net MUX_S1: U10.11 (S1), U6.11 (S1), U7.11 (S1), U8.11 (S1), U9.11 (S1)
- new net MUX_S2: U10.14 (S2), U6.14 (S2), U7.14 (S2), U8.14 (S2), U9.14 (S2)
- new net MUX_S3: U10.13 (S3), U6.13 (S3), U7.13 (S3), U8.13 (S3), U9.13 (S3)

Commit message: pcb updated
Parts:
- HE42: footprint PCM_marbastlib-xp-he:SW_MX_HE_90deg_1u_Rules -> PCM_marbastlib-xp-he:SW_MX_HE_90deg_2.25u_Rules
Connections:
- net HE54_Shift is gone; now on net HE54_RShift: HE55.2 (VOUT)
- net HE67_Up is gone; now on net HE67_Right: HE68.2 (VOUT)
- net GND: now also U8.17 (I14), U8.18 (I13), U8.20 (I11), U8.21 (I10), U8.4 (I5), U8.7 (I2), U8.9 (I0), U9.22 (I9), U9.4 (I5), U9.6 (I3), U9.7 (I2), U9.9 (I0)
- net HE0_Esc: now also U6.21 (I10)
- net HE10_0: now also U9.3 (I6)
- net HE11_Minus: now also U10.21 (I10)
- net HE12_Equal: now also U10.22 (I9)
- net HE13_Backspace: now also U10.2 (I7)
- net HE14_Tab: now also U6.20 (I11)
- net HE15_Q: now also U6.23 (I8)
- net HE16_W: now also U6.3 (I6)
- net HE17_E: now also U6.6 (I3)
- net HE18_R: now also U7.21 (I10)
- net HE19_T: now also U7.4 (I5)
- net HE1_1: now also U6.22 (I9)
- net HE20_Y: now also U7.7 (I2)
- net HE21_U: now also U8.23 (I8)
- net HE22_I: now also U9.21 (I10)
- net HE23_O: now also U9.5 (I4)
- net HE24_P: now also U9.2 (I7)
- net HE25_LeftBracket: now also U10.20 (I11)
- net HE26_RightBracket: now also U10.23 (I8)
- net HE27_Backslash: now also U10.3 (I6)
- net HE28_Delete: now also U10.4 (I5)
- net HE29_CapsLock: now also U6.19 (I12)
- net HE2_2: now also U6.2 (I7)
- net HE30_A: now also U6.7 (I2)
- net HE31_S: now also U7.20 (I11)
- net HE32_D: now also U7.19 (I12)
- net HE33_F: now also U7.22 (I9)
- net HE34_G: now also U7.3 (I6)
- net HE35_H: now also U8.22 (I9)
- net HE36_J: now also U8.2 (I7)
- net HE37_K: now also U8.5 (I4)
- net HE38_L: now also U9.17 (I14)
- net HE39_Semicolon: now also U9.8 (I1)
- net HE3_3: now also U6.4 (I5)
- net HE40_Quote: now also U10.19 (I12)
- net HE41_Enter: now also U10.9 (I0)
- net HE42_PgUp: now also U10.5 (I4)
- net HE43_Shift: now also U6.18 (I13)
- net HE44_Z: now also U6.8 (I1)
- net HE45_X: now also U7.18 (I13)
- net HE46_C: now also U7.17 (I14)
- net HE47_V: now also U7.23 (I8)
- net HE48_B: now also U7.9 (I0)
- net HE49_N: now also U8.16 (I15)
- net HE4_4: now also U6.5 (I4)
- net HE50_M: now also U8.8 (I1)
- net HE51_Comma: now also U8.6 (I3)
- net HE52_Period: now also U9.16 (I15)
- net HE53_Slash: now also U9.20 (I11)
- net HE55_Up: now also U10.8 (I1)
- net HE56_PgDn: now also U10.6 (I3)
- net HE57_Ctrl: now also U6.17 (I14)
- net HE58_Win: now also U6.16 (I15)
- net HE59_LAlt: now also U6.9 (I0)
- net HE5_5: now also U7.2 (I7)
- net HE60_Space: now also U7.16 (I15)
- net HE61_Space2: now also U7.8 (I1)
- net HE62_Space3: now also U8.19 (I12)
- net HE63_RAlt: now also U9.19 (I12)
- net HE64_Fn: now also U9.18 (I13)
- net HE65_Left: now also U10.17 (I14)
- net HE66_Down: now also U10.18 (I13)
- net HE6_6: now also U7.5 (I4)
- net HE7_7: now also U7.6 (I3)
- net HE8_8: now also U8.3 (I6)
- net HE9_9: now also U9.23 (I8)
- net HE54_RShift: now reaches U10.16 (I15)
- net HE67_Right: now reaches U10.7 (I2)
